Commit message: Major change in the use of URDF links with fixed joints to apply forces and torques

File: gym_pybullet_drones/assets/cf2p.urdf (robot description, URDF)
Before this commit: robot cf2, 1 links, 0 joints
Links:
- added link center_of_mass_link, mass 0
- added link prop0_link, mass 0
- added link prop1_link, mass 0
- added link prop2_link, mass 0
- added link prop3_link, mass 0
Joints:
- added joint center_of_mass_joint: type fixed, parent base_link, child center_of_mass_link
- added joint prop0_joint: type fixed, parent base_link, child prop0_link
- added joint prop1_joint: type fixed, parent base_link, child prop1_link
- added joint prop2_joint: type fixed, parent base_link, child prop2_link
- added joint prop3_joint: type fixed, parent base_link, child prop3_link

File: gym_pybullet_drones/assets/cf2x.urdf (robot description, URDF)
Before this commit: robot cf2, 1 links, 0 joints
Links:
- added link center_of_mass_link, mass 0
- added link prop0_link, mass 0
- added link prop1_link, mass 0
- added link prop2_link, mass 0
- added link prop3_link, mass 0
Joints:
- added joint center_of_mass_joint: type fixed, parent base_link, child center_of_mass_link
- added joint prop0_joint: type fixed, parent base_link, child prop0_link
- added joint prop1_joint: type fixed, parent base_link, child prop1_link
- added joint prop2_joint: type fixed, parent base_link, child prop2_link
- added joint prop3_joint: type fixed, parent base_link, child prop3_link

File: gym_pybullet_drones/assets/hb.urdf (robot description, URDF)
Before this commit: robot quad, 1 links, 0 joints
Links:
- added link center_of_mass_link, mass 0
- added link prop0_link, mass 0
- added link prop1_link, mass 0
- added link prop2_link, mass 0
- added link prop3_link, mass 0
Joints:
- added joint center_of_mass_joint: type fixed, parent base_link, child center_of_mass_link
- added joint prop0_joint: type fixed, parent base_link, child prop0_link
- added joint prop1_joint: type fixed, parent base_link, child prop1_link
- added joint prop2_joint: type fixed, parent base_link, child prop2_link
- added joint prop3_joint: type fixed, parent base_link, child prop3_link
