Commit message: c++ trajectory generation almost working

File: gym_pybullet_drones/assets/simple_tree.urdf (robot description, URDF)
Before this commit: robot simple_tree, 2 links, 1 joints
Links:
- link canopy: geometry collision sphere radius=1.0; visual sphere radius=1.0
- link trunk: geometry collision cylinder length=2.0 radius=0.2; visual cylinder length=2.0 radius=0.2
